File: X17_Backplane.kicad_sch (KiCad schematic)
At the start: 5 parts, among them J1 CLT-110-01-F-D, J3 HTST-110-04-L-D-RA, J4 ET60S-D04-3-08-D04-X-R1-S, J5 IPT1-105-01-L-D, J7 IPT1-105-01-L-D

Commit message: Work done on 10/9/24
Connections:
- net 5V is gone; now on net P07: J1.01, J1.03
- net GNDRAT is gone; now on net P05: J1.02, J1.04, J5.NC@1*6 (NC), J7.NC@1*6 (NC)
- net P06 is gone; now on net P05: J4.P06_1 (P06)
- net P08 is gone; now on net P07: J4.P08_1 (P08)
- net A: now reaches J1.05
- net B: now reaches J1.07
Other:
- moved on the sheet: J7

Commit message: Work on 10/12/24
Parts:
- removed J3: HTST-110-04-L-D-RA, CONN_HTST-110-04/05-x-D-RA_SAI, symbol 2024-10-03_15-47-29:HTST-110-04-L-D-RA
- added J2: DF11-10DS-2DSA05, CON10_2X5_U_DF11_MOL_HIR, symbol DF11_10DS_2DSA_05_:DF11-10DS-2DSA05
- added J3, J8: 430450212, CON_430450212_MOL, symbol 430450212:430450212
- added J9: HTST-110-04-L-D-RA, CONN_HTST-110-04/05-x-D-RA_SAI, symbol 2024-10-03_15-47-29:HTST-110-04-L-D-RA
- added U1: ~, symbol DF11_10DS_2DSA_05_:DF11-10DS-2DSA05v2
Connections:
- net A: now also J2.3, J3.1
- net B: now also J2.4, J3.2
- net P05: no longer J1.02, J1.04, J4.P06_1 (P06), J5.NC@1*6 (NC), J7.NC@1*6 (NC)
- net P07: no longer J1.01, J1.03, J4.P08_1 (P08)
- net PWMA0: now also J2.7
- net PWMA1: now also J2.8
- net PWMA2: now also J2.9
- net PWMA3: now also J2.10
- net PWMB0: now also U1.13
- net PWMB1: now also U1.14
- net PWMB2: now also U1.15
- net PWMB3: now also U1.16
- net PWMC0: now also U1.17
- net PWMC1: now also U1.18
- net PWMC2: now also U1.19
- net PWMC3: now also U1.20
- new net 5V: J1.01, J1.03, J2.1, J2.2, J8.1
- new net 5V_GND: J1.02, J1.04, J8.2
- new net GNDRAT: J5.NC@1*6 (NC), J7.NC@1*6 (NC)
- new net P06: J4.P06_1 (P06)
- new net P08: J4.P08_1 (P08)

Commit message: Final Work 10/12/2024
Parts:
- removed J1: CLT-110-01-F-D, CLT-110-01-F-D:SAMTEC_CLT-110-01-F-D, symbol CLT-110-01-F-D:CLT-110-01-F-D
- removed J2: DF11-10DS-2DSA05, CON10_2X5_U_DF11_MOL_HIR, symbol DF11_10DS_2DSA_05_:DF11-10DS-2DSA05
- removed J3, J8: 430450212, CON_430450212_MOL, symbol 430450212:430450212
- removed J4: ET60S-D04-3-08-D04-X-R1-S, ET60S-D04-3-08-D04-X-R1-S:SAMTEC_ET60S-D04-3-08-D04-X-R1-S, symbol ET60S-D04-3-08-D04-X-R1-S:ET60S-D04-3-08-D04-X-R1-S
- removed J5, J7: IPT1-105-01-L-D, IPT1-105-01-L-D:SAMTEC_IPT1-105-01-L-D, symbol IPT1-105-01-L-D:IPT1-105-01-L-D
- removed J9: HTST-110-04-L-D-RA, CONN_HTST-110-04/05-x-D-RA_SAI, symbol 2024-10-03_15-47-29:HTST-110-04-L-D-RA
- removed U1: ~, symbol DF11_10DS_2DSA_05_:DF11-10DS-2DSA05v2
Other:
- added sheet Connectors (Connectors.kicad_sch)
- note removed: "ESC ADAPTER CONNECTIONS"
- note removed: "ESC CONTROLLER CONNECTOR"
- note removed: "PI SHIELD CONNECTOR"
- note removed: "POWER SLAB CONNECTOR"

Commit message: Work done on 10/16/2024
Other:
- added sheet LEDS&PWR (LEDS&PWR.kicad_sch)
Changed lines of the file:
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@@
 	(paper "A4")
+	(sheet
+		(at 72.39 21.59)
+		(size 27.94 21.59)
+		(fields_autoplaced yes)
+		(stroke
+			(width 0.1524)
+			(type solid)
+		)
+		(fill
+			(color 0 0 0 0.0000)
+		)
+		(property "Sheetname" "LEDS&PWR"
+			(at 72.39 20.8784 0)
+			(effects
+				(font
+					(size 1.27 1.27)
+				)
+				(justify left bottom)
+			)
+		)
+		(property "Sheetfile" "LEDS&PWR.kicad_sch"
+			(at 72.39 43.7646 0)
+			(effects
+				(font
+					(size 1.27 1.27)
+				)
+				(justify left top)
+			)
+		)
+		(instances
+			(project "X17_Backplane"
+				(path "/0b609d63-053d-4947-8bc2-b53c83cfcb53"
+					(page "3")
+				)
+			)
+		)
+	)
 	(sheet
 		(at 24.13 22.86)
