File: Connectors.kicad_sch (KiCad schematic)
At the start: 14 parts, among them J1 430450212, J11 430450212, J12 DF11-10DS-2DSA05, J14 ET60S-D04-3-08-D04-X-R1-S, J2 IPS1-105-01-L-D, J3 IPS1-105-01-L-D, J4 Conn_01x02_Pin, J5 Conn_01x04_Pin, J8 430450612

Commit message: Work done after office hours on 10/20/24
Parts:
- added J6: Conn_01x02_Pin, symbol Connector:Conn_01x02_Pin
Connections:
- net A_TB: now also J6.1 (Pin_1)
- net B_TB: now also J6.2 (Pin_2)
- net CS: now also J5.4 (Pin_4)
- net MISO: now also J5.1 (Pin_1)
- net MOSI: now also J5.2 (Pin_2)
- net SCLK: now also J5.3 (Pin_3)
- no-connect marks 29 -> 31
Other:
- note added: "TOOL'S BOARD OUTPUT"
Changed lines of the file:
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@@
+	)
+	(no_connect
+		(at 45.72 146.05)
 	)
 	(no_connect
@@
 	(no_connect
 		(at 217.17 57.15)
+	)
+	(no_connect
+		(at 45.72 138.43)
 	)
 	(no_connect
@@
 		)
 	)
+	(text "TOOL'S BOARD OUTPUT"
+		(exclude_from_sim no)
+		(at 131.826 94.234 0)
+		(effects
+			(font
+				(size 1.27 1.27)
+			)
+		)
+	)
 	(text "ESC CONTROLLER CONNECTOR "
 		(exclude_from_sim no)
@@
 		)
 	)
+	(global_label "CS"
+		(shape input)
+		(at 161.29 78.74 0)
+		(fields_autoplaced yes)
+		(effects
+			(font
+				(size 0.762 0.762)
+			)
+			(justify left)
+		)
+		(property "Intersheetrefs" "${INTERSHEET_REFS}"
+			(at 164.5691 78.74 0)
+			(effects
+				(font
+					(size 1.27 1.27)
+				)
+				(justify left)
+				(hide yes)
+			)
+		)
+	)
 	(global_label "12V_1"
 		(shape input)
@@
 		)
 	)
+	(global_label "MOSI"
+		(shape input)
+		(at 161.29 73.66 0)
+		(fields_autoplaced yes)
+		(effects
+			(font
+				(size 0.762 0.762)
+			)
+			(justify left)
+		)
+		(property "Intersheetrefs" "${INTERSHEET_REFS}"
+			(at 165.8392 73.66 0)
+			(effects
+				(font
+					(size 1.27 1.27)
+				)
+				(justify left)
+				(hide yes)
+			)
+		)
+	)
 	(global_label "5V_GND"
 		(shape input)
@@
 		)
 	)
+	(global_label "A_TB"
+		(shape input)
+		(at 135.89 102.87 0)
+		(fields_autoplaced yes)
+		(effects
+			(font
+				(size 0.762 0.762)
+			)
+			(justify left)
+		)
+		(property "Intersheetrefs" "${INTERSHEET_REFS}"
+			(at 140.2577 102.87 0)
+			(effects
+				(font
+					(size 1.27 1.27)
+				)
+				(justify left)
+				(hide yes)
+			)
+		)
+	)
 	(global_label "PWMA1"
 		(shape input)
@@
 		)
 	)
+	(global_label "B_TB"
+		(shape input)
+		(at 135.89 105.41 0)
+		(fields_autoplaced yes)
+		(effects
+			(font
+				(size 0.762 0.762)
+			)
+			(justify left)
+		)
+		(property "Intersheetrefs" "${INTERSHEET_REFS}"
+			(at 140.3666 105.41 0)
+			(effects
+				(font
+					(size 1.27 1.27)
+				)
+				(justify left)
+				(hide yes)
+			)
+		)
+	)
 	(global_label "PWMA2"
 		(shape input)
@@
 		)
 	)
+	(global_label "SCLK"
+		(shape input)
+		(at 161.29 76.2 0)
+		(fields_autoplaced yes)
+		(effects
+			(font
+				(size 0.762 0.762)
+			)
+			(justify left)
+		)
+		(property "Intersheetrefs" "${INTERSHEET_REFS}"
+			(at 165.948 76.2 0)
+			(effects
+				(font
+					(size 1.27 1.27)
+				)
+				(justify left)
+				(hide yes)
+			)
+		)
+	)
 	(global_label "PWMA3"
 		(shape input)
@@
 		)
 	)
+	(global_label "MISO"
+		(shape input)
+		(at 161.29 71.12 0)
+		(fields_autoplaced yes)
+		(effects
+			(font
+				(size 0.762 0.762)
+			)
+			(justify left)
+		)
+		(property "Intersheetrefs" "${INTERSHEET_REFS}"
+			(at 165.8392 71.12 0)
+			(effects
+				(font
+					(size 1.27 1.27)
+				)
+				(justify left)
+				(hide yes)
+			)
+		)
+	)
 	(global_label "Telemetry"
 		(shape input)
@@
 			)
 		)
+	)
+	(symbol
+		(lib_id "Connector:Conn_01x02_Pin")
+		(at 130.81 102.87 0)
+		(unit 1)
+		(exclude_from_sim no)
+		(in_bom yes)
+		(on_board yes)
+		(dnp no)
+		(fields_autoplaced yes)
+		(property "Reference" "J6"
+			(at 131.445 97.79 0)
+			(effects
+				(font
+					(size 1.27 1.27)
+				)
+			)
+		)
+		(property "Value" "Conn_01x02_Pin"
+			(at 131.445 100.33 0)
+			(effects
+				(font
+					(size 1.27 1.27)
+				)
+			)
+		)
+		(property "Footprint" ""
+			(at 130.81 102.87 0)
+			(effects
+				(font
+					(size 1.27 1.27)
+				)
+				(hide yes)
+			)
+		)
+		(property "Datasheet" "~"
+			(at 130.81 102.87 0)
+			(effects
+				(font
+					(size 1.27 1.27)
+				)
+				(hide yes)
+			)
+		)
+		(property "Description" "Generic connector, single row, 01x02, script generated"
+			(at 130.81 102.87 0)
+			(effects
+				(font
+					(size 1.27 1.27)
+				)
+				(hide yes)
+			)
+		)
+		(pin "2"
+		)
+		(pin "1"
+		)
+		(instances
+			(project ""
+				(path "/0b609d63-053d-4947-8bc2-b53c83cfcb53/ad869c69-8d32-4ec0-b8bb-9dda93ac11ca"
+					(reference "J6")
+					(unit 1)
+				)
+			)
+		)

Commit message: Work done on 10/23/2024
Parts:
- removed J6: Conn_01x02_Pin, symbol Connector:Conn_01x02_Pin
- added U1: 282837-4, 282837-4_TYC, symbol 2024-10-23_23-38-15:282837-4
- R1, R2, R3, R4: value R_US -> 10K
Connections:
- net 5V is gone; now on net P05: J12.1, J8.1, R1.1, R3.1
- net 5V_GND is gone; now on net P06: J12.2, J8.2, R2.2, R4.2
- net A_TB: now also U1.4
- net B_TB: now also U1.3
- net P07: now also U1.1
- net P08: now also U1.2
- no-connect marks 31 -> 27

Commit message: Updates on 10/24/2024
Parts:
- removed J11: 430450212, CON_430450212_MOL, symbol 430450212:430450212
Connections:
- net A: now also J8.4
- net B: now also J8.3
- net NRST: now also J8.6; no longer J8.5
- net NRST2: now also J8.5; no longer J8.4
- net P05: now also R2.2; no longer R1.1
- net P06: now also R1.1; no longer R2.2
- no-connect marks 27 -> 25
Other:
- moved on the sheet: J8

Commit message: Update 10/25/2024 (again lol)
Connections:
- net P05: now also R4.2; no longer R3.1
- net P06: now also R3.1; no longer R4.2

Commit message: Work done on 10/30/2024
Parts:
- removed R1, R2, R3, R4: 10K, symbol Device:R_US
- J1: footprint CON_430450212_MOL -> CON430450612:CON_430450612_MOL
- J12: footprint CON10_2X5_U_DF11_MOL_HIR -> DF11_10DS_2DSA:CON10_2X5_U_DF11_MOL_HIR
- J2, J3: footprint IPS1-105-01-L-D:SAMTEC_IPS1-105-01-L-D -> IPS1_105_01_L_D_RA:SAMTEC_IPS1-105-01-L-D-RA
- J4: footprint (none) -> Connector_PinHeader_1.00mm:PinHeader_1x02_P1.00mm_Vertical
- J5: footprint (none) -> Connector_PinHeader_1.00mm:PinHeader_1x04_P1.00mm_Vertical
- J8: footprint CON_430450612_MOL -> 430450612:CON_430450612_MOL
- U1: footprint 282837-4_TYC -> 282837_3footprints:282837-3_TYC
- U2: footprint (none) -> DF11_10DS_2DSA:CON10_2X5_U_DF11_MOL_HIR

Commit message: Work on 10/31/2024
Parts:
- removed U2: ~, DF11_10DS_2DSA:CON10_2X5_U_DF11_MOL_HIR, symbol DF11_10DS_2DSA_05_:DF11-10DS-2DSA05v2
- added J17: DF11-10DS-2DSA05, DF11_10DS_2DSA:CON10_2X5_U_DF11_MOL_HIR, symbol DF11_10DS_2DSA_05_:DF11-10DS-2DSA05
- J1: footprint CON430450612:CON_430450612_MOL -> 430450212:CON_430450212_MOL
Connections:
- net CS: now also J17.10
- net MISO: now also J17.7
- net MOSI: now also J17.8
- net NRST: now also J17.6
- net PWMB2: now also J17.1
- net PWMB3: now also J17.2
- net PWMC0: now also J17.3
- net PWMC1: now also J17.4
- net SCLK: now also J17.9
- net Telemetry: now also J17.5

Commit message: Work on 11/2/2024
Parts:
- added J18: 430450212, CON_430450212_MOL, symbol 430450212:430450212
- added U2: ULN2003AD, D0016A_N, symbol ULN2003AD:ULN2003AD
- J12, J17: footprint DF11_10DS_2DSA:CON10_2X5_U_DF11_MOL_HIR -> DF11_10DS_2SA_05:CON10_2X5_UF_DF11_HIR
- U1: footprint 282837_3footprints:282837-3_TYC -> TB_282837_4:282837-4_TYC
Connections:
- net A: now also J18.2; no longer J8.4
- net B: now also J18.1; no longer J8.3
- net P01: now also U2.9 (COM)
- net P02: now also U2.8 (GND)
- new net 5V_GNDTB: J8.4
- new net 5V_TB: J8.3
- new net GPIO1: U2.1 (IN1)
- new net GPIO2: U2.2 (IN2)
- new net GPIO3: U2.3 (IN3)
- new net GPIO4: U2.4 (IN4)
- new net GPIO5: U2.5 (IN5)
- new net GPIO6: U2.6 (IN6)
- new net GPIO7: U2.7 (IN7)
- new net SOL1_1: U2.16 (OUT1)
- new net SOL2_1: U2.15 (OUT2)
- new net SOL3_1: U2.14 (OUT3)
- new net SOL4_1: U2.13 (OUT4)
- new net SOL5_1: U2.12 (OUT5)
- new net SOL6_1: U2.11 (OUT6)
- new net SOL7_1: U2.10 (OUT7)
Other:
- moved on the sheet: J1, J8, U1

Commit message: Work done on 11/06/2024
Parts:
- added U3: SolenoidConn, SolenoidFootPrint:PXC-8-RA-1778683, symbol SolenoidConn:SolConn
- J18: footprint CON_430450212_MOL -> 430450212:CON_430450212_MOL
- U2: footprint D0016A_N -> ul_ULN2003ADfootprints:D0016A_L
Connections:
- net A: now also J14.17; no longer J14.19
- net B: now also J14.18; no longer J14.20
- net NRST2: now also J14.19; no longer J14.21
- net P02: now also U3.1, U3.2
- net P05: no longer J12.1, J8.1
- net P06: no longer J12.2, J8.2
- net P07: no longer U1.1
- net P08: no longer U1.2
- net SOL1_1: now also U3.8
- net SOL2_1: now also U3.7
- net SOL3_1: now also U3.6
- net SOL4_1: now also U3.5
- net SOL5_1: now also U3.4
- net SOL6_1: now also U3.3
- net 48V: now reaches J14.01
- net 48V: now also J14.02, U1.1
- net 48V_GND: now reaches J14.22
- net 48V_GND: now also J14.23, U1.2
- new net 5V: J12.1, J14.20, J8.1
- new net 5V_GND: J12.2, J14.21, J8.2
- no-connect marks 25 -> 23
Other:
- note added: "SOLENOID STUFF"
