File: Connectors.kicad_sch (KiCad schematic)
At the start: 13 parts, among them J1 430450212, J12 DF11-10DS-2DSA05, J14 ET60S-D04-3-08-D04-X-R1-S, J17 DF11-10DS-2DSA05, J18 430450212, J2 IPS1-105-01-L-D, J3 IPS1-105-01-L-D, J4 Conn_01x02_Pin, J5 Conn_01x04_Pin, J8 430450612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

Commit message: Work done on 11/09/2024
Parts:
- removed J12, J17: DF11-10DS-2DSA05, DF11_10DS_2SA_05:CON10_2X5_UF_DF11_HIR, symbol DF11_10DS_2DSA_05_:DF11-10DS-2DSA05
- added J19: DF11-10DS-2DSA05, DF11_10_DP_2DSA:CON10_2X5_UF_DF11_HIR, symbol DF11_10DS_2DSA_05_:DF11-10DS-2DSA05
- J2, J3: footprint IPS1_105_01_L_D_RA:SAMTEC_IPS1-105-01-L-D-RA -> ESCadapterfootprint:PWM, 12V, GND JST Connector
Connections:
- net 5V: now also J19.1
- net 5V_GND: now also J19.2
- net A: now also J19.3
- net B: now also J19.4
- net CS: now also J19.20
- net MISO: now also J19.17
- net MOSI: now also J19.18
- net NRST: now also J19.16
- net PWMA0: now also J19.5
- net PWMA1: now also J19.6
- net PWMA2: now also J19.7
- net PWMA3: now also J19.8
- net PWMB0: now also J19.9
- net PWMB1: now also J19.10
- net PWMB2: now also J19.11
- net PWMB3: now also J19.12
- net PWMC0: now also J19.13
- net PWMC1: now also J19.14
- net SCLK: now also J19.19
- net Telemetry: now also J19.15
Other:
- moved on the sheet: J4, J5

Commit message: Work done on 11/12/2024
Parts:
- J2, J3: footprint ESCadapterfootprint:PWM, 12V, GND JST Connector -> ESCadapterfootprint:PWM, 12V, GND JST Connector (1)
Changed lines of the file:
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@@
 			)
 		)
-		(property "Footprint" "ESCadapterfootprint:PWM, 12V, GND JST Connector"
+		(property "Footprint" "ESCadapterfootprint:PWM, 12V, GND JST Connector (1)"
 			(at 44.45 60.96 0)
 			(effects
@@
 			)
 		)
-		(property "Footprint" "ESCadapterfootprint:PWM, 12V, GND JST Connector"
+		(property "Footprint" "ESCadapterfootprint:PWM, 12V, GND JST Connector (1)"
 			(at 44.45 38.1 0)
 			(effects

Commit message: Work done on 11/14/2024
Connections:
- net P06 is gone; now on net P05: J14.P06_1 (P06)
- net P08 is gone; now on net P07: J14.P08_1 (P08)
- net A: now also J14.01; no longer J14.17
- net B: now also J14.02; no longer J14.18
- net NRST2: now also J14.03; no longer J14.19
- net P01: now also J2.02, J2.03, U2.8 (GND), U3.1, U3.2; no longer J2.01, U2.9 (COM)
- net P02: now also J3.02, J3.03; no longer J2.02, J2.03, U2.8 (GND), U3.1, U3.2
- net P03: now also J2.01, U2.9 (COM); no longer J3.01
- net P04: now also J3.01; no longer J3.02, J3.03
- net P05: now also U1.2
- net P07: now also U1.1
- removed net 48V: J14.01, J14.02, U1.1
- removed net 48V_GND: J14.22, J14.23, U1.2

Commit message: Work done on11/17/2024
I'm cooked yo
Parts:
- removed U1: 282837-4, TB_282837_4:282837-4_TYC, symbol 2024-10-23_23-38-15:282837-4
- added U1: 282837-6, 282837_6:282837-6_TYC, symbol 282837_6:282837-6
Connections:
- net 5V_GNDTB: now also J8.6, U1.6; no longer J8.4
- net P05: no longer J14.P06_1 (P06)
- net P07: no longer J14.P08_1 (P08)
- net 48V: now reaches J14.05
- net 48V: now also J14.06, U1.2
- net 48V_GND: now reaches J14.07
- net 48V_GND: now also J14.08, U1.1
- net 5V_TB renamed NRST_PSB
- net NRST_PSB: now also J14.03
- net A renamed A+
- net A_TB renamed A_TB+
- net A_TB+: now also U1.4
- net B renamed A-
- net B_TB renamed A_TB-
- net A_TB-: now also U1.5
- net NRST renamed NRST_ESCC
- net NRST_ESCC: now also J8.4; no longer J8.6
- net NRST2 renamed NRST_TB
- net NRST_TB: now also U1.3; no longer J14.03
- new net P06: J14.P06_1 (P06)
- new net P08: J14.P08_1 (P08)

Commit message: WORK done on 11/20/2024
I'm losing my shiiiiiii
#SlayedTheDayAway
Connections:
- net A+: now also J19.4; no longer J19.3
- net A-: now also J19.6; no longer J19.4
- net PWMA1: now also J19.3; no longer J19.6

Commit message: Work done on 11/22/2024
Parts:
- removed J4: Conn_01x02_Pin, Connector_PinHeader_1.00mm:PinHeader_1x02_P1.00mm_Vertical, symbol Connector:Conn_01x02_Pin
- removed J5: Conn_01x04_Pin, Connector_PinHeader_1.00mm:PinHeader_1x04_P1.00mm_Vertical, symbol Connector:Conn_01x04_Pin
- added J20, J21, J22, J23, J4, J5: Conn_01x01, TestPoint:TestPoint_Pad_D4.0mm, symbol Connector_Generic:Conn_01x01
- J2, J3: footprint ESCadapterfootprint:PWM, 12V, GND JST Connector (1) -> ESCadapterfootprint:PWM, 12V, GND JST Connector (real)
Connections:
- net 48V: now also U1.5; no longer U1.2
- net 48V_GND: now also U1.4; no longer U1.1
- net A+: now also J4.1 (Pin_1)
- net A-: now also J5.1 (Pin_1)
- net A_TB+: now also U1.2; no longer U1.4
- net A_TB-: now also U1.3; no longer U1.5
- net CS: now also J21.1 (Pin_1)
- net MISO: now also J22.1 (Pin_1)
- net MOSI: now also J23.1 (Pin_1)
- net NRST_TB: now also U1.1; no longer U1.3
- net SCLK: now also J20.1 (Pin_1)
Other:
- note added: "RS485 Test Point"
- note added: "SPI Test Point"

Commit message: Work done on 12/13/2024
Parts:
- removed J20, J21, J22, J23, J4, J5: Conn_01x01, TestPoint:TestPoint_Pad_D4.0mm, symbol Connector_Generic:Conn_01x01
- added J4: Conn_01x04_Pin, Connector_PinHeader_2.54mm:PinHeader_1x04_P2.54mm_Vertical_SMD_Pin1Right, symbol Connector:Conn_01x04_Pin
- added J6: Conn_01x02_Pin, Connector_PinHeader_2.54mm:PinHeader_1x02_P2.54mm_Vertical, symbol Connector:Conn_01x02_Pin
Connections:
- net 48V: now also J14.21, J14.22; no longer J14.05, J14.06
- net 48V_GND: now also J14.23, J14.24; no longer J14.07, J14.08
- net 5V: now also J14.19; no longer J14.20
- net 5V_GND: now also J14.20; no longer J14.21
- net A+: now also J6.1 (Pin_1)
- net A-: now also J6.2 (Pin_2)
- net CS: now also J4.4 (Pin_4)
- net MISO: now also J4.1 (Pin_1)
- net MOSI: now also J4.2 (Pin_2)
- net P01: no longer J2.02, J2.03, U2.8 (GND), U3.1, U3.2
- net P02: no longer J3.02, J3.03
- net P03: no longer J2.01, U2.9 (COM)
- net P04: no longer J3.01
- net P05: now also J2.01, J3.01, U2.9 (COM)
- net P08: now also J2.02, J2.03, J3.02, J3.03, U2.8 (GND), U3.1, U3.2
- net SCLK: now also J4.3 (Pin_3)
- no-connect marks 23 -> 25

Commit message: Work done on 12/14/2024
Parts:
- J4: footprint Connector_PinHeader_2.54mm:PinHeader_1x04_P2.54mm_Vertical_SMD_Pin1Right -> Connector_PinHeader_2.54mm:PinHeader_1x04_P2.54mm_Vertical
- U3: footprint SolenoidFootPrint:PXC-8-RA-1778683 -> Connector_PinHeader_2.54mm:PinHeader_1x08_P2.54mm_Vertical
Connections:
- net P08: no longer U3.2
- net SOL7_1: now also U3.2
Changed lines of the file:
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@@
 	(generator_version "8.0")
 	(paper "A4")
-	(junction
-		(at 100.33 154.94)
-		(diameter 0)
-		(color 0 0 0 0)
-	)
 	(no_connect
 		(at 217.17 67.31)
@@
 	(wire
 		(pts
-			(xy 100.33 152.4) (xy 100.33 154.94)
+			(xy 55.88 105.41) (xy 59.69 105.41)
 		)
 		(stroke
@@
 		)
 	)
-	(wire
-		(pts
-			(xy 100.33 157.48) (xy 104.14 157.48)
-		)
-		(stroke
-			(width 0)
-			(type default)
-		)
-	)
-	(wire
-		(pts
-			(xy 100.33 154.94) (xy 104.14 154.94)
-		)
-		(stroke
-			(width 0)
-			(type default)
-		)
-	)
-	(wire
-		(pts
-			(xy 100.33 154.94) (xy 100.33 157.48)
-		)
-		(stroke
-			(width 0)
-			(type default)
-		)
-	)
-	(wire
-		(pts
-			(xy 55.88 105.41) (xy 59.69 105.41)
-		)
-		(stroke
-			(width 0)
-			(type default)
-		)
-	)
 	(text "PI SHIELD CONNECTOR "
 		(exclude_from_sim no)
@@
 	(global_label "12V_GND"
 		(shape input)
-		(at 100.33 152.4 180)
-		(fields_autoplaced yes)
-		(effects
-			(font
-				(size 0.762 0.762)
-			)
-			(justify right)
-		)
-		(property "Intersheetrefs" "${INTERSHEET_REFS}"
-			(at 93.5312 152.4 0)
+		(at 104.14 154.94 180)
+		(fields_autoplaced yes)
+		(effects
+			(font
+				(size 0.762 0.762)
+			)
+			(justify right)
+		)
+		(property "Intersheetrefs" "${INTERSHEET_REFS}"
+			(at 97.3412 154.94 0)
 			(effects
 				(font
@@
 		(property "Intersheetrefs" "${INTERSHEET_REFS}"
 			(at 119.6569 34.29 0)
+			(effects
+				(font
+					(size 1.27 1.27)
+				)
+				(justify right)
+				(hide yes)
+			)
+		)
+	)
+	(global_label "SOL7_1"
+		(shape input)
+		(at 104.14 157.48 180)
+		(fields_autoplaced yes)
+		(effects
+			(font
+				(size 0.762 0.762)
+			)
+			(justify right)
+		)
+		(property "Intersheetrefs" "${INTERSHEET_REFS}"
+			(at 98.1757 157.48 0)
 			(effects
 				(font
@@
 			)
 		)
-		(property "Footprint" "Connector_PinHeader_2.54mm:PinHeader_1x04_P2.54mm_Vertical_SMD_Pin1Right"
+		(property "Footprint" "Connector_PinHeader_2.54mm:PinHeader_1x04_P2.54mm_Vertical"
 			(at 156.21 74.93 0)
 			(effects
@@
 			)
 		)
-		(property "Footprint" "SolenoidFootPrint:PXC-8-RA-1778683"
+		(property "Footprint" "Connector_PinHeader_2.54mm:PinHeader_1x08_P2.54mm_Vertical"
 			(at 104.14 152.4 0)
 			(effects
