File: X17_Backplane.kicad_pcb (KiCad board)
At the start: 2 copper layers, 89.2 x 110 mm, 0 parts

Commit message: Work done on 10/30/2024
Parts:
- added C2: 180μF, Capacitor_SMD:C_0805_2012Metric, F.Cu at (102.6, 118.6)
- added C5: 180μF, Capacitor_SMD:C_0805_2012Metric, F.Cu at (102.6, 121.6)
- added D1: LED, LED_SMD:LED_0805_2012Metric, F.Cu at (102.7, 106.5)
- added D2: LED, LED_SMD:LED_0805_2012Metric, F.Cu at (102.7, 109.5)
- added D3: LED, LED_SMD:LED_0805_2012Metric, F.Cu at (102.7, 112.5)
- added D4: LED, LED_SMD:LED_0805_2012Metric, F.Cu at (102.7, 115.6)
- added J1: 430450212, CON430450612:CON_430450612_MOL, F.Cu at (142.5, 79.2)
- added J10: Conn_01x01, Connector_PinHeader_1.00mm:PinHeader_1x01_P1.00mm_Vertical, F.Cu at (96.1, 115.6)
- added J11: Conn_01x01, Connector_PinHeader_1.00mm:PinHeader_1x01_P1.00mm_Vertical, F.Cu at (96.1, 118.7)
- added J12: DF11-10DS-2DSA05, DF11_10DS_2DSA:CON10_2X5_U_DF11_MOL_HIR, F.Cu at (105.3, 80.4)
- added J13: Conn_01x01, Connector_PinHeader_1.00mm:PinHeader_1x01_P1.00mm_Vertical, F.Cu at (96.1, 121.7)
- added J14: ET60S-D04-3-08-D04-X-R1-S, ET60S-D04-3-08-D04-X-R1-S:SAMTEC_ET60S-D04-3-08-D04-X-R1-S, F.Cu at (138.0, 50.7)
- added J15: Conn_01x01, Connector_PinHeader_1.00mm:PinHeader_1x01_P1.00mm_Vertical, F.Cu at (96.1, 124.8)
- added J16: Conn_01x01, Connector_PinHeader_1.00mm:PinHeader_1x01_P1.00mm_Vertical, F.Cu at (96.1, 127.8)
- added J2: IPS1-105-01-L-D, IPS1_105_01_L_D_RA:SAMTEC_IPS1-105-01-L-D-RA, F.Cu at (123.2, 73.8)
- added J3: IPS1-105-01-L-D, IPS1_105_01_L_D_RA:SAMTEC_IPS1-105-01-L-D-RA, F.Cu at (123.2, 88.6)
- added J4: Conn_01x02_Pin, Connector_PinHeader_1.00mm:PinHeader_1x02_P1.00mm_Vertical, F.Cu at (129.8, 114.8)
- added J5: Conn_01x04_Pin, Connector_PinHeader_1.00mm:PinHeader_1x04_P1.00mm_Vertical, F.Cu at (126.4, 114.8)
- added J6: Conn_01x01, Connector_PinHeader_1.00mm:PinHeader_1x01_P1.00mm_Vertical, F.Cu at (96.1, 106.5)
- added J7: Conn_01x01, Connector_PinHeader_1.00mm:PinHeader_1x01_P1.00mm_Vertical, F.Cu at (96.1, 109.5)
- added J8: 430450612, 430450612:CON_430450612_MOL, F.Cu at (142.5, 91.7)
- added J9: Conn_01x01, Connector_PinHeader_1.00mm:PinHeader_1x01_P1.00mm_Vertical, F.Cu at (96.1, 112.6)
- added R5: 600, Resistor_SMD:R_0805_2012Metric, F.Cu at (107.1, 106.4)
- added R6: 250, Resistor_SMD:R_0805_2012Metric, F.Cu at (107.1, 109.4)
- added R7: 600, Resistor_SMD:R_0805_2012Metric, F.Cu at (107.1, 112.3)
- added R8: 4K, Resistor_SMD:R_0805_2012Metric, F.Cu at (107.1, 115.3)
- added U1: 282837-4, 282837_3footprints:282837-3_TYC, F.Cu at (152.8, 76.0)
- added U2: ~, DF11_10DS_2DSA:CON10_2X5_U_DF11_MOL_HIR, F.Cu at (105.3, 96.3)

Commit message: Work on 10/31/2024
Parts:
- removed U2: ~, DF11_10DS_2DSA:CON10_2X5_U_DF11_MOL_HIR
- added J17: DF11-10DS-2DSA05, DF11_10DS_2DSA:CON10_2X5_U_DF11_MOL_HIR, F.Cu at (136.5, 103.3)
- J1: footprint CON430450612:CON_430450612_MOL -> 430450212:CON_430450212_MOL
- moved J1 64.3 mm to (171.2, 136.8)
- moved C2 59.7 mm to (147.7, 79.3)
- moved C5 59.7 mm to (147.7, 82.3)
- moved D1 59.7 mm to (147.7, 67.2)
- moved D2 59.7 mm to (147.7, 70.2)
- moved D3 59.7 mm to (147.7, 73.2)
- moved D4 59.7 mm to (147.7, 76.3)
- moved J10 59.7 mm to (141.2, 76.3)
- moved J11 59.7 mm to (141.2, 79.4)
- moved J13 59.7 mm to (141.2, 82.4)
- moved J15 59.7 mm to (141.2, 85.5)
- moved J16 59.7 mm to (141.2, 88.5)
- moved J6 59.7 mm to (141.2, 67.2)
- moved J7 59.7 mm to (141.2, 70.2)
- moved J9 59.7 mm to (141.2, 73.3)
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
Commit message: Work on 11/2/2024
Parts:
- J12, J17: footprint DF11_10DS_2DSA:CON10_2X5_U_DF11_MOL_HIR -> DF11_10DS_2SA_05:CON10_2X5_UF_DF11_HIR
- U1: footprint 282837_3footprints:282837-3_TYC -> TB_282837_4:282837-4_TYC
- moved J12 3.09 mm to (136.0, 51.1)
- moved J14 1.51 mm to (101.8, 95.5)

Commit message: Work done on 11/06/2024
Parts:
- added J18: 430450212, 430450212:CON_430450212_MOL, F.Cu at (127.8, 95.2)
- added U2: ULN2003AD, ul_ULN2003ADfootprints:D0016A_L, F.Cu at (143.8, 52.9)
- added U3: SolenoidConn, SolenoidFootPrint:PXC-8-RA-1778683, F.Cu at (115.8, 45.0)
- moved J3 91.6 mm to (159.0, 45.3)
- moved J12 83.8 mm to (141.0, 134.8), turned to 90 degrees
- moved D1 78.3 mm to (69.8, 59.4)
- moved D2 78.3 mm to (69.8, 62.5)
- moved D3 78.3 mm to (69.8, 65.5)
- moved D4 78.3 mm to (69.8, 68.5)
- moved J10 78.3 mm to (63.2, 68.6)
- moved J11 78.3 mm to (63.2, 71.6)
- moved J13 78.3 mm to (63.2, 74.7)
- moved J6 78.3 mm to (63.2, 59.4)
- moved J7 78.3 mm to (63.2, 62.5)
- moved J9 78.3 mm to (63.2, 65.5)
- moved R5 78.3 mm to (74.2, 59.4)
- moved R6 78.3 mm to (74.2, 62.3)
- moved R7 78.3 mm to (74.2, 65.3)
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Connections:
- D4 pad 2: 24V -> 48V
- J11 pad 1: 24V_GND -> 48V_GND
- J14 pad 01: unconnected-(J14-Pad01) -> 48V
- J14 pad 02: unconnected-(J14-Pad02) -> 48V
- J14 pad 17: unconnected-(J14-Pad17) -> A
- J14 pad 18: unconnected-(J14-Pad18) -> B
- J14 pad 19: A -> NRST2
- J14 pad 20: B -> 5V
- J14 pad 21: NRST2 -> 5V_GND
- J14 pad 22: unconnected-(J14-Pad22) -> 48V_GND
- J14 pad 23: unconnected-(J14-Pad23) -> 48V_GND
- J14 pad P05_1: 5V -> P05
- J14 pad P06_1: 5V_GND -> P06
- J14 pad P07_1: 24V -> P07
- J14 pad P08_1: 24V_GND -> P08
- J6 pad 1: 24V -> 48V
- J8 pad 3: B -> 5V_TB
- J8 pad 4: A -> 5V_GNDTB
- R8 pad 2: 24V_GND -> 48V_GND
- U1 pad 1: 24V -> 48V
- U1 pad 2: 24V_GND -> 48V_GND
Routing:
- added copper zone on F.Cu, net 12V_1
- added copper zone on F.Cu, net 12V_2
- added copper zone on F.Cu, net 12V_GND1
- added copper zone on F.Cu, net 12V_GND2

Commit message: Work done on 11/09/2024
Parts:
- removed J12, J17: DF11-10DS-2DSA05, DF11_10DS_2SA_05:CON10_2X5_UF_DF11_HIR
- added J19: DF11-10DS-2DSA05, DF11_10_DP_2DSA:CON10_2X5_UF_DF11_HIR, F.Cu at (231.3, 147.0)
- J2, J3: footprint IPS1_105_01_L_D_RA:SAMTEC_IPS1-105-01-L-D-RA -> ESCadapterfootprint:PWM, 12V, GND JST Connector
- moved R5 190.9 mm to (257.7, 111.8)
- moved R6 190.9 mm to (257.7, 114.8)
- moved R7 190.9 mm to (257.7, 117.7)
- moved R8 190.9 mm to (257.7, 120.7)
- moved C2 190.9 mm to (253.2, 124.0)
- moved C5 190.9 mm to (253.2, 127.0)
- moved D1 190.9 mm to (253.2, 111.9)
- moved D2 190.9 mm to (253.2, 114.9)
- moved D3 190.9 mm to (253.2, 118.0)
- moved D4 190.9 mm to (253.2, 121.0)
- moved J10 190.9 mm to (246.7, 121.0)
- moved J11 190.9 mm to (246.7, 124.1)
- moved J13 190.9 mm to (246.7, 127.1)
- moved J6 190.9 mm to (246.7, 111.9)
- moved J7 190.9 mm to (246.7, 114.9)
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Connections:
- net P05 renamed P05_7
- net P06 renamed P06_6
- net P07 renamed P07_8
- net P08 renamed P08_6
Routing:
- removed copper zone on F.Cu, net 12V_1
- removed copper zone on F.Cu, net 12V_2
- removed copper zone on F.Cu, net 12V_GND1
- removed copper zone on F.Cu, net 12V_GND2

Commit message: Work done on 11/12/2024
Parts:
- J2, J3: footprint ESCadapterfootprint:PWM, 12V, GND JST Connector -> ESCadapterfootprint:PWM, 12V, GND JST Connector (1)
- moved J2 41.4 mm to (145.8, 81.7), turned to 90 degrees
- moved J3 27.7 mm to (164.5, 81.8), turned to 90 degrees
Routing:
- added copper zone on F.Cu, net 12V_1
- added copper zone on F.Cu, net 12V_2
- added copper zone on B.Cu, net 12V_GND1
- added copper zone on F.Cu, net 12V_GND2

Commit message: Work done 11/13/2024
Parts:
- moved J19 85.1 mm to (147.0, 135.0)
- moved J8 29.0 mm to (134.7, 145.2)
- moved J3 12.9 mm to (177.5, 82.0), turned to -90 degrees
- turned J2 to -90 degrees
Routing:
- net 5V: track 0.00 -> 150.0 mm
- net A: track 0.00 -> 89.1 mm
- net B: track 0.00 -> 68.1 mm, vias 0 -> 2
- net 5V_GND: track 0.00 -> 60.1 mm
- added copper zone on B.Cu, net 12V_GND2
- removed copper zone on F.Cu, net 12V_GND2

Commit message: Work done on 11/14/2024
Parts:
- moved J2 2.78 mm to (143.0, 81.8)
- moved J19 2.01 mm to (148.0, 136.8)
- moved J14 0.93 mm to (101.0, 95.0)
- moved J3 0.17 mm to (177.5, 82.2)
Connections:
- J14 pad 01: 48V -> A
- J14 pad 02: 48V -> B
- J14 pad 03: unconnected-(J14-Pad03) -> NRST2
- J14 pad 17: A -> unconnected-(J14-Pad17)
- J14 pad 18: B -> unconnected-(J14-Pad18)
- J14 pad 19: NRST2 -> unconnected-(J14-Pad19)
- J14 pad 22: 48V_GND -> unconnected-(J14-Pad22)
- J14 pad 23: 48V_GND -> unconnected-(J14-Pad23)
- J14 pad P01_1: 12V_1 -> 12V_GND1
- J14 pad P02_1: 12V_GND1 -> 12V_GND2
- J14 pad P03_1: 12V_2 -> 12V_1
- J14 pad P04_1: 12V_GND2 -> 12V_2
- J14 pad P05_1: P05_7 -> 48V_GND
- J14 pad P06_1: P06_6 -> 48V_GND
- J14 pad P07_1: P07_8 -> 48V
- J14 pad P08_1: P08_6 -> 48V
Routing:
- net 5V: track 150.0 -> 0.00 mm
- net A: track 89.1 -> 0.00 mm
- net B: track 68.1 -> 0.00 mm, vias 2 -> 0
- net 5V_GND: track 60.1 -> 0.00 mm
- added copper zone on F.Cu, net 12V_GND1
- added copper zone on F.Cu, net 12V_GND2
- removed copper zone on B.Cu, net 12V_GND1
- removed copper zone on B.Cu, net 12V_GND2
