File: X17_Backplane.kicad_pcb (KiCad board)
At the start: 2 copper layers, 89.2 x 110 mm, 25 parts, among them J1 430450212, J14 ET60S-D04-3-08-D04-X-R1-S, J15 Conn_01x01, J16 Conn_01x01, J18 430450212, J19 DF11-10DS-2DSA05, J2 IPS1-105-01-L-D, J3 IPS1-105-01-L-D, J4 Conn_01x01, J4 Conn_01x04_Pin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

Commit message: Work done on 12/14/2024
Parts:
- U3: footprint SolenoidFootPrint:PXC-8-RA-1778683 -> Connector_PinHeader_2.54mm:PinHeader_1x08_P2.54mm_Vertical
- moved U3 0.56 mm to (166.8, 87.6), turned to 180 degrees
Connections:
- U3 pad 2: 12V_GND -> SOL7_1
Routing:
- net PWMA1: track 0.00 -> 77.9 mm
- net PWMA0: track 0.00 -> 69.8 mm
- net PWMA2: track 0.00 -> 67.4 mm, vias 0 -> 2
- net 5V: track 1.97 -> 68.9 mm, vias 0 -> 2
- net PWMB2: track 0.00 -> 58.5 mm
- net PWMB0: track 0.00 -> 46.0 mm, vias 0 -> 4
- net PWMB1: track 0.00 -> 44.0 mm, vias 0 -> 2
- net PWMB3: track 0.00 -> 43.0 mm
- net 12V_GND: track 118.9 -> 140.3 mm, vias 3 -> 4
- net 5V_GND: track 0.00 -> 21.4 mm, vias 0 -> 2
- net Telemetry: track 0.00 -> 17.9 mm
- net PWMA3: track 0.00 -> 17.6 mm
- net 12V: track 126.8 -> 139.2 mm, vias 3 -> 4
- net SOL7_1: track 0.00 -> 12.0 mm
- net SOL1_1: track 0.00 -> 11.7 mm
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- added copper zone on B.Cu, net 5V_GND

Commit message: More work done on 12/14/2024
Parts:
- moved 5V_GND 78.4 mm to (110.6, 88.8)
- moved R6 66.1 mm to (127.0, 112.6)
- moved D2 66.0 mm to (127.0, 107.8)
- moved 5V 65.3 mm to (118.2, 108.0)
- moved J6 60.8 mm to (99.8, 143.5)
- renumbered J15 to 5V, J16 to 5V_GND
Routing:
- net 12V_GND: track 140.3 -> 163.6 mm, vias 4 -> 5
- net 5V_GND: track 21.4 -> 36.8 mm, vias 2 -> 3
- net A+: track 0.00 -> 13.2 mm
- net A-: track 1.20 -> 12.5 mm
- net 5V: track 68.9 -> 79.3 mm
- net Net-(D2-K): track 0.00 -> 2.86 mm
Changed lines of the file:
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@@
 	(footprint "Resistor_SMD:R_0603_1608Metric_Pad0.98x0.95mm_HandSolder"
 		(layer "F.Cu")
-		(at 68.0334 142.45 -90)
+		(at 127 112.6 -90)
 		(descr "Resistor SMD 0603 (1608 Metric), square (rectangular) end terminal, IPC_7351 nominal with elongated pad for handsoldering. (Body size source: IPC-SM-782 page 72, https://www.pcb-3d.com/wordpress/wp-content/uploads/ipc-sm-782a_amendment_1_and_2.pdf), generated with kicad-footprint-generator")
 		(tags "resistor handsolder")
@@
 	(footprint "Connector_PinHeader_2.54mm:PinHeader_1x02_P2.54mm_Vertical"
 		(layer "F.Cu")
-		(at 74 88.46)
+		(at 99.8 143.525)
 		(descr "Through hole straight pin header, 1x02, 2.54mm pitch, single row")
 		(tags "Through hole pin header THT 1x02 2.54mm single row")
@@
 	(footprint "LED_SMD:LED_0805_2012Metric_Pad1.15x1.40mm_HandSolder"
 		(layer "F.Cu")
-		(at 68.0334 137.45 90)
+		(at 127 107.8 90)
 		(descr "LED SMD 0805 (2012 Metric), square (rectangular) end terminal, IPC_7351 nominal, (Body size source: https://docs.google.com/spreadsheets/d/1BsfQQcO9C6DZCsRaXUlFlo91Tg2WpOkGARC1WS5S8t0/edit?usp=sharing), generated with kicad-footprint-generator")
 		(tags "LED handsolder")
@@
 	(footprint "TestPoint:TestPoint_Pad_D4.0mm"
 		(layer "F.Cu")
-		(at 78.2834 159.7)
+		(at 118.2 108)
 		(descr "SMD pad as test Point, diameter 4.0mm")
 		(tags "test point SMD pad")
-		(property "Reference" "J15"
-			(at -3.25 -1.75 0)
+		(property "Reference" "5V"
+			(at -3.6 -0.2 0)
 			(layer "F.SilkS")
 			(effects
@@
 	(footprint "TestPoint:TestPoint_Pad_D4.0mm"
 		(layer "F.Cu")
-		(at 83.7834 162.45)
+		(at 110.6 88.8)
 		(descr "SMD pad as test Point, diameter 4.0mm")
 		(tags "test point SMD pad")
-		(property "Reference" "J16"
-			(at 0 -2.898 0)
+		(property "Reference" "5V_GND"
+			(at 2.2 -3.2 0)
 			(layer "F.SilkS")
 			(effects
@@
 	)
 	(segment
+		(start 171.2 86.4)
+		(end 177 80.6)
+		(width 0.889)
+		(layer "F.Cu")
+		(net 1)
+	)
+	(segment
+		(start 169.96 87.64)
+		(end 171.2 86.4)
+		(width 0.889)
+		(layer "F.Cu")
+		(net 1)
+	)
+	(segment
+		(start 177 80.6)
+		(end 177 72.4)
+		(width 0.889)
+		(layer "F.Cu")
+		(net 1)
+	)
+	(segment
+		(start 166.8 87.64)
+		(end 169.96 87.64)
+		(width 0.889)
+		(layer "F.Cu")
+		(net 1)
+	)
+	(segment
+		(start 177 72.4)
+		(end 177 70.4)
+		(width 0.889)
+		(layer "F.Cu")
+		(net 1)
+	)
+	(segment
 		(start 149.786 82.2)
 		(end 142.8 75.214)
@@
 	)
 	(via
+		(at 177 70.4)
+		(size 0.6)
+		(drill 0.3)
+		(layers "F.Cu" "B.Cu")
+		(net 1)
+	)
+	(via
 		(at 142.8 65.2)
 		(size 0.6)
@@
 	)
 	(segment
-		(start 149.999999 109.000001)
-		(end 142.4 109.000001)
+		(start 113.6 100)
+		(end 115 100)
 		(width 0.889)
 		(layer "F.Cu")
@@
 	)
 	(segment
-		(start 113.6 100)
-		(end 115 100)
+		(start 127 105)
+		(end 128.2 103.8)
 		(width 0.889)
 		(layer "F.Cu")
@@
 	)
 	(segment
-		(start 151 103.8)
-		(end 151.8 104.6)
+		(start 127 106.775)
+		(end 127 105)
+		(width 0.889)
+		(layer "F.Cu")
+		(net 4)
+	)
+	(segment
+		(start 151.8 104.6)
+		(end 151.8 107.2)
 		(width 0.889)
 		(layer "F.Cu")
@@
 	)
 	(segment
-		(start 151.8 104.6)
-		(end 151.8 107.2)
+		(start 108.6 99.8)
+		(end 107.39 98.59)
+		(width 0.889)
+		(layer "F.Cu")
+		(net 4)
+	)
+	(segment
+		(start 91.533401 160.633683)
+		(end 91.533401 160.95)
+		(width 0.508)
+		(layer "F.Cu")
+		(net 4)
+	)
+	(segment
+		(start 122.4 103.8)
+		(end 123.4 103.8)
 		(width 0.889)
 		(layer "F.Cu")
@@
 	)
 	(segment
-		(start 108.6 99.8)
-		(end 107.39 98.59)
+		(start 128.2 103.8)
+		(end 151 103.8)
 		(width 0.889)
 		(layer "F.Cu")
@@
 	)
 	(segment
-		(start 91.533401 160.633683)
-		(end 91.533401 160.95)
-		(width 0.508)
+		(start 151 103.8)
+		(end 151.8 104.6)
+		(width 0.889)
+		(layer "F.Cu")
+		(net 4)
+	)
+	(segment
+		(start 123.4 103.8)
+		(end 128.2 103.8)
+		(width 0.889)
+		(layer "F.Cu")
+		(net 4)
+	)
+	(segment
+		(start 118.2 108)
+		(end 122.4 103.8)
+		(width 0.889)
+		(layer "F.Cu")
+		(net 4)
+	)
+	(segment
+		(start 149.999999 109.000001)
+		(end 142.4 109.000001)
+		(width 0.889)
 		(layer "F.Cu")
 		(net 4)
@@
 	(segment
 		(start 118.8 103.8)
-		(end 151 103.8)
+		(end 123.4 103.8)
 		(width 0.889)
 		(layer "F.Cu")
@@
 	)
 	(segment
+		(start 127 108.825)
+		(end 127 111.6875)
+		(width 0.889)
+		(layer "F.Cu")
+		(net 5)
+	)
+	(segment
 		(start 125.9 124.9)
 		(end 128.91 124.9)
@@
 	)
 	(segment
-		(start 108.65 96.05)
+		(start 112 97.4)
+		(end 110.65 96.05)
+		(width 0.889)
+		(layer "F.Cu")
+		(net 20)
+	)
+	(segment
+		(start 110.65 96.05)
 		(end 100.08 96.05)
 		(width 0.889)
@@
 	)
 	(segment
-		(start 111.2 98.6)
-		(end 108.65 96.05)
+		(start 112 107)
+		(end 112 97.4)
+		(width 0.889)
+		(layer "F.Cu")
+		(net 20)
+	)
+	(segment
+		(start 127 113.5125)
+		(end 127 115.6)
+		(width 0.889)
+		(layer "F.Cu")
+		(net 20)
+	)
+	(segment
+		(start 107.8 96.05)
+		(end 110.6 93.25)
 		(width 0.889)
 		(layer "F.Cu")
@@
 	)
 	(segment
-		(start 111.2 103.6)
-		(end 111.2 98.6)
+		(start 110.6 93.25)
+		(end 110.6 88.8)
 		(width 0.889)
 		(layer "F.Cu")
@@
 	)
 	(via
-		(at 111.2 103.6)
+		(at 112 107)
 		(size 0.6)
 		(drill 0.3)
@@
 		(net 20)
 	)
+	(via
+		(at 127 115.6)
+		(size 0.6)
+		(drill 0.3)
+		(layers "F.Cu" "B.Cu")
+		(net 20)
+	)
 	(segment
 		(start 162.99 78.39)
@@
 	)
 	(segment
+		(start 111 143.200001)
+		(end 108.450002 145.749999)
+		(width 0.2)
+		(layer "F.Cu")
+		(net 69)
+	)
+	(segment
+		(start 102.024999 145.749999)
+		(end 99.8 143.525)
+		(width 0.2)
+		(layer "F.Cu")
+		(net 69)
+	)
+	(segment
+		(start 108.450002 145.749999)
+		(end 102.024999 145.749999)
+		(width 0.2)
+		(layer "F.Cu")
+		(net 69)
+	)
+	(segment
+		(start 111 146.2)
+		(end 101.838603 146.2)
+		(width 0.2)
+		(layer "F.Cu")
+		(net 70)
+	)
+	(segment
+		(start 101.703603 146.065)
+		(end 99.8 146.065)
+		(width 0.2)
+		(layer "F.Cu")
+		(net 70)
+	)
+	(segment
+		(start 101.838603 146.2)
+		(end 101.703603 146.065)
+		(width 0.2)
+		(layer "F.Cu")
+		(net 70)
+	)
+	(segment
 		(start 73.9334 150.55)
 		(end 74.7834 149.7)
@@
 		(polygon
 			(pts
-				(xy 94.8 76.6) (xy 94.8 83.2) (xy 113.6 83.2) (xy 113.6 97.4) (xy 125 97.4) (xy 125 102.2) (xy 134.4 102.2)
+				(xy 94.8 76.6) (xy 94.8 83.2) (xy 116.6 83.2) (xy 116.6 97.4) (xy 125 97.4) (xy 125 102.2) (xy 134.4 102.2)
 				(xy 134.4 96.4) (xy 173.6 96.6) (xy 173.6 102.4) (xy 181.6 102.4) (xy 181.6 85.8) (xy 173.6 85.8)
-				(xy 173.6 91.2) (xy 134.6 91) (xy 134.6 85.8) (xy 125 85.8) (xy 125 91) (xy 120.4 91) (xy 120.4 76.6)
+				(xy 173.6 91.2) (xy 134.6 91) (xy 134.6 85.8) (xy 125 85.8) (xy 125 91.2) (xy 122.6 91.2) (xy 122.6 76.8)
 			)
 		)
@@
 		(polygon
 			(pts
-				(xy 91.68 101.67) (xy 91.6 152.4) (xy 182.6 152.2) (xy 182.8 102.8)
+				(xy 91.28 104.87) (xy 91.6 152.4) (xy 182.6 152.2) (xy 182.4 106)
 			)
 		)

Commit message: Work done on 12/16/2024
Parts:
- removed the J4 at (74.3, 142.7)
- removed the J4 at (108.9, 167.7)
- removed J5: Conn_01x01, TestPoint:TestPoint_Pad_D4.0mm
- added J4: Conn_01x07_Pin, Connector_PinHeader_2.54mm:PinHeader_1x07_P2.54mm_Vertical, F.Cu at (146.1, 87.4)
- moved 12V 57.2 mm to (170.6, 83.6)
- moved R5 37.3 mm to (176.1, 75.0)
- moved D1 37.3 mm to (176.1, 80.6)
- moved J8 32.5 mm to (113.5, 117.4), turned to 180 degrees
- moved U3 14.6 mm to (162.7, 73.6), turned to -90 degrees
- moved U2 2.42 mm to (153.8, 80.2), turned to 90 degrees
- renumbered J7 to 12V, 5V to J15, 5V_GND to J16
Connections:
- J19 pad 17: MISO -> unconnected-(J19-Pad17)
- J19 pad 18: MOSI -> unconnected-(J19-Pad18)
- J19 pad 19: SCLK -> unconnected-(J19-Pad19)
- J19 pad 20: CS -> unconnected-(J19-Pad20)
Routing:
- net NRST_ESCC: track 0.00 -> 83.0 mm, vias 0 -> 2
- net Telemetry: track 17.9 -> 87.7 mm, vias 0 -> 2
- net NRST_PSB: track 0.00 -> 44.8 mm
- net 12V_GND: track 163.6 -> 135.3 mm, vias 5 -> 4
- net PWMB2: track 58.5 -> 46.8 mm
- net GPIO7: track 0.00 -> 8.39 mm
- net SOL5_1: track 10.9 -> 4.20 mm
- net GPIO6: track 0.00 -> 6.69 mm
- net GPIO1: track 0.00 -> 6.66 mm
- net SOL4_1: track 10.4 -> 4.23 mm
- net GPIO2: track 0.00 -> 6.02 mm
- net SOL6_1: track 11.5 -> 5.54 mm
- net PWMB3: track 43.0 -> 37.1 mm
- net SOL3_1: track 10.6 -> 4.99 mm
- net 5V_GND: track 36.8 -> 42.2 mm, vias 3 -> 4
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Other:
- board text removed: "A+"
- board text removed: "A-"
- board text removed: "D1"

Commit message: Work done on 12/16/2024 v2
Parts:
- moved J6 78.4 mm to (178.2, 141.3)
- moved J18 57.2 mm to (167.2, 135.3), turned to -90 degrees
- moved U1 55.3 mm to (97.7, 143.5)
- moved J15 44.3 mm to (73.9, 107.0)
- moved R6 29.5 mm to (154.7, 102.4), turned to 0 degrees
- moved D2 22.2 mm to (148.6, 102.5), turned to 180 degrees
- moved J1 3.36 mm to (142.2, 142.4), turned to 180 degrees
- renumbered 12V to J7
Connections:
- J14 pad 01: A+ -> A-
- J14 pad 02: A- -> A+
- J19 pad 17: unconnected-(J19-Pad17) -> A+
- J19 pad 18: unconnected-(J19-Pad18) -> A-
Routing:
- net A-: track 11.3 -> 107.8 mm
- net A+: track 13.2 -> 106.0 mm
- net A_TB+: track 0.00 -> 46.6 mm
- net A_TB-: track 0.00 -> 41.6 mm
- net NRST_TB: track 0.00 -> 40.6 mm
- net 5V_GNDTB: track 0.00 -> 24.6 mm
- net 5V_GND: track 42.2 -> 48.5 mm
- net PWMB1: track 44.7 -> 49.3 mm, vias 2 -> 4
- net NRST_ESCC: track 83.0 -> 86.3 mm, vias 2 -> 4
- net 5V: track 79.4 -> 77.4 mm
- net PWMA3: track 17.6 -> 15.8 mm
- net Net-(D2-K): track 2.86 -> 4.20 mm
- net Telemetry: track 87.7 -> 88.3 mm, vias 2 -> 4
- net PWMB2: track 46.8 -> 46.6 mm, vias 0 -> 2
- net PWMB3: track 37.1 -> 36.9 mm, vias 0 -> 2
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
Commit message: Work done on 12/17/2024
Parts:
- added C1: 180μF, EEE_FT1E561UPfootprints:CAP_FT_F_PAN, F.Cu at (170.6, 78.4)
- 12V LED: renamed from D1
- 5V GND: renamed from J16
- 5V LED: renamed from D2
- 600 : renamed from R5
- moved 5V GND 89.1 mm to (178.1, 146.9)
- moved R8 86.0 mm to (111.0, 87.2), turned to 90 degrees
- moved 48V 80.2 mm to (111.0, 91.7), turned to -90 degrees
- moved 5V 52.7 mm to (126.5, 109.5)
- moved J4 43.9 mm to (148.3, 43.6)
- moved 12VGND 37.1 mm to (142.5, 77.4)
- moved U2 29.9 mm to (155.4, 50.3), turned to -90 degrees
- moved J6 24.7 mm to (160.4, 124.2), turned to 90 degrees
- moved 600  23.5 mm to (152.6, 76.0)
- moved 12V LED 23.5 mm to (152.6, 81.4)
- moved U3 22.6 mm to (148.0, 56.4), turned to 90 degrees
- moved 12V 11.6 mm to (159.0, 84.3)
- moved J18 6.27 mm to (161.7, 132.3), turned to 90 degrees
- renumbered J7 to 12V, J9 to 12VGND, D4 to 48V, J15 to 5V
Connections:
- J14 pad 01: A- -> Aout-
- J14 pad 02: A+ -> Aout+
- J19 pad 4: A+ -> Aout+
- J19 pad 6: A- -> Aout-
- J4 pad 1: GPIO1 -> GPIO7
- J4 pad 2: GPIO2 -> GPIO6
- J4 pad 3: GPIO3 -> GPIO5
- J4 pad 5: GPIO5 -> GPIO3
- J4 pad 6: GPIO6 -> GPIO2
- J4 pad 7: GPIO7 -> GPIO1
Routing:
- net 48V: track 0.31 -> 82.2 mm
- net 48V_GND: track 0.00 -> 76.4 mm
- net 12V: track 138.3 -> 210.4 mm, vias 5 -> 20
- net A-: track 107.8 -> 42.1 mm
- net Aout+: track 0.00 -> 65.7 mm
- net Aout-: track 0.00 -> 64.2 mm
- net A+: track 106.0 -> 47.1 mm
- net 12V_GND: track 135.3 -> 189.4 mm, vias 4 -> 31
- net PWMB3: track 36.9 -> 84.3 mm, vias 2 -> 0
- net PWMB2: track 46.6 -> 91.4 mm, vias 2 -> 0
- net Telemetry: track 88.3 -> 129.9 mm, vias 4 -> 2
- net PWMB1: track 49.3 -> 84.0 mm, vias 4 -> 2
- net PWMB0: track 48.0 -> 61.1 mm, vias 4 -> 2
- net 5V: track 77.4 -> 85.5 mm
- net 5V_GND: track 48.5 -> 43.3 mm, vias 4 -> 5
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Other:
- board text added: "TEST"
- board text added: "X17 Backplane Vijay, Daniel, Leo, Keona Vishakh"

Commit message: Work on 12/17/2024 v2
Routing:
- net A-: track 42.1 -> 40.1 mm
- net A_TB+: track 46.6 -> 45.8 mm

Commit message: work on 12/17/2024 v3
Routing:
- net NRST_PSB: track 45.1 -> 46.0 mm

Commit message: Work done on 12/17/2024 final
Am i done??????
Parts:
- added J5: Conn_01x01_Pin, Connector_PinHeader_2.54mm:PinHeader_1x01_P2.54mm_Vertical, F.Cu at (108.5, 47.1)
- added PWMC: Conn_01x01_Pin, Connector_PinHeader_2.54mm:PinHeader_1x01_P2.54mm_Vertical, F.Cu at (175.9, 106.4)
- added RS485: Conn_01x02_Pin, Connector_PinHeader_2.54mm:PinHeader_1x02_P2.54mm_Vertical, F.Cu at (144.8, 142.8)
- added U4: 282837-3, 282837_3footprints:282837-3_TYC, F.Cu at (115.0, 47.5)
- 12V GND: renamed from 12VGND
- moved J1 7.60 mm to (134.6, 142.5)
- moved 5V 3.23 mm to (129.6, 108.3)
- renumbered R6 to 250, R8 to 4K, J6 to RS485
Connections:
- J14 pad P01_1: P01_9 -> (no net)
- J14 pad P02_1: P02_4 -> (no net)
- J14 pad P03_1: P03_8 -> (no net)
- J14 pad P04_1: P04_9 -> (no net)
- J14 pad P06_1: P06_7 -> 12V
- J14 pad P07_1: P07_4 -> 12V_GND
Routing:
- net 12V: track 210.4 -> 296.7 mm, vias 20 -> 18
- net 12V_GND: track 189.4 -> 268.7 mm, vias 31 -> 29
- net Aout-: track 64.7 -> 52.5 mm
- net Aout+: track 65.5 -> 53.3 mm
- net PWMC0: track 0.00 -> 9.66 mm
- net PWMC0_OUT: track 0.00 -> 6.71 mm
- net 5V_GND: track 43.3 -> 47.5 mm
- net A_TB+: track 45.8 -> 49.4 mm
- net A_TB-: track 41.6 -> 44.5 mm
- net 5V: track 85.4 -> 86.3 mm
Other:
- board text added: "PWMC"
- board text added: "TB"
