File: LEDS&PWR.kicad_sch (KiCad schematic)
At the start: 6 parts

Commit message: Work done on 10/19/2024
Parts:
- removed C1, C2, C3, C4, C5, C6: 560μF, CAP_FT_F_PAN, symbol P122427CT-ND:EEE-FT1E561UP
- added C1, C2, C3, C4, C5, C6: 180μF, CAP_FN_F_PAN, symbol 2024-10-19_19-04-44:EEE-FN1H181UP
- added D1, D2, D3: LED, symbol Device:LED
- added R5, R6, R7: R_US, symbol Device:R_US
Connections:
- net 12V_1: now also C1.1, C2.1, C3.1, D1.2 (A)
- net 12V_2: now also C4.1, C5.1, C6.1, D3.2 (A)
- net 12V_GND1: now also C1.2, C2.2, C3.2, R5.2
- net 12V_GND2: now also C4.2, C5.2, C6.2, R7.2
- new net: D3.1 (K), R7.1
- new net: D2.1 (K), R6.1
- new net: D1.1 (K), R5.1
- new net 5V: D2.2 (A)
- new net 5V_GND: R6.2
Other:
- note added: "12V LED"
- note added: "5V CAPACITORS"
- note added: "5V LED"

Commit message: Work done after office hours on 10/20/24
Parts:
- removed C1, C3, C4, C6: 180μF, CAP_FN_F_PAN, symbol 2024-10-19_19-04-44:EEE-FN1H181UP
- added J10, J13, J15, J16, J7, J9: Conn_01x01, symbol Connector_Generic:Conn_01x01
- R5, R7: value R_US -> 600
- R6: value R_US -> 250
Connections:
- net 12V_GND2 is gone; now on net GNDPWR: C5.2, R7.2
- net 12V_1: now also J7.1 (Pin_1)
- net 12V_2: now also J10.1 (Pin_1)
- net 5V: now also J15.1 (Pin_1)
- net 5V_GND: now also J16.1 (Pin_1)
- net 12V_GND1 renamed GNDPWR
- net GNDPWR: now also J13.1 (Pin_1), J9.1 (Pin_1)
Other:
- note added: "POWER TEST POINTS"
- note added: "PWR FLAGS"
- note removed: "5V CAPACITORS"

Commit message: Work done on 10/23/2024
Connections:
- net GNDPWR renamed 12V_GND1
- net 12V_GND1: no longer C5.2, J13.1 (Pin_1), R7.2
- new net 12V_GND2: C5.2, J13.1 (Pin_1), R7.2
Other:
- moved on the sheet: C2, C5, D1, D2, D3, R5, R6, R7

Commit message: Updates on 10/24/2024
Parts:
- added D4: LED, symbol Device:LED
- added J11, J6: Conn_01x01, symbol Connector_Generic:Conn_01x01
- added R8: 4K, symbol Device:R_US
Connections:
- net 24V: now also D4.2 (A), J6.1 (Pin_1)
- net 24V_GND: now also J11.1 (Pin_1), R8.2
- new net: D4.1 (K), R8.1
Other:
- note added: "24V LED"
- moved on the sheet: J10, J13, J15, J16, J7, J9

Commit message: Work done on 10/30/2024
Parts:
- C2, C5: footprint CAP_FN_F_PAN -> Capacitor_SMD:C_0805_2012Metric
- D1, D2, D3, D4: footprint (none) -> LED_SMD:LED_0805_2012Metric
- J10, J11, J13, J15, J16, J6, J7, J9: footprint (none) -> Connector_PinHeader_1.00mm:PinHeader_1x01_P1.00mm_Vertical
- R5, R6, R7, R8: footprint (none) -> Resistor_SMD:R_0805_2012Metric
Changed lines of the file:
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@@
 			)
 		)
-		(property "Footprint" ""
+		(property "Footprint" "LED_SMD:LED_0805_2012Metric"
 			(at 121.92 33.02 0)
 			(effects
@@
 			)
 		)
-		(property "Footprint" ""
+		(property "Footprint" "Connector_PinHeader_1.00mm:PinHeader_1x01_P1.00mm_Vertical"
 			(at 114.3 107.95 0)
 			(effects
@@
 			)
 		)
-		(property "Footprint" "CAP_FN_F_PAN"
+		(property "Footprint" "Capacitor_SMD:C_0805_2012Metric"
 			(at 44.45 39.37 0)
 			(effects
@@
 			)
 		)
-		(property "Footprint" ""
+		(property "Footprint" "Connector_PinHeader_1.00mm:PinHeader_1x01_P1.00mm_Vertical"
 			(at 114.3 95.25 0)
 			(effects
@@
 			)
 		)
-		(property "Footprint" ""
+		(property "Footprint" "LED_SMD:LED_0805_2012Metric"
 			(at 171.45 30.48 0)
 			(effects
@@
 			)
 		)
-		(property "Footprint" ""
+		(property "Footprint" "Connector_PinHeader_1.00mm:PinHeader_1x01_P1.00mm_Vertical"
 			(at 114.3 119.38 0)
 			(effects
@@
 			)
 		)
-		(property "Footprint" "CAP_FN_F_PAN"
+		(property "Footprint" "Capacitor_SMD:C_0805_2012Metric"
 			(at 30.48 39.37 0)
 			(effects
@@
 			)
 		)
-		(property "Footprint" ""
+		(property "Footprint" "Connector_PinHeader_1.00mm:PinHeader_1x01_P1.00mm_Vertical"
 			(at 114.3 88.9 0)
 			(effects
@@
 			)
 		)
-		(property "Footprint" ""
+		(property "Footprint" "Connector_PinHeader_1.00mm:PinHeader_1x01_P1.00mm_Vertical"
 			(at 114.3 132.08 0)
 			(effects
@@
 			)
 		)
-		(property "Footprint" ""
+		(property "Footprint" "Resistor_SMD:R_0805_2012Metric"
 			(at 94.996 44.704 90)
 			(effects
@@
 			)
 		)
-		(property "Footprint" ""
+		(property "Footprint" "LED_SMD:LED_0805_2012Metric"
 			(at 93.98 33.02 0)
 			(effects
@@
 			)
 		)
-		(property "Footprint" ""
+		(property "Footprint" "LED_SMD:LED_0805_2012Metric"
 			(at 227.33 34.29 0)
 			(effects
@@
 			)
 		)
-		(property "Footprint" ""
+		(property "Footprint" "Resistor_SMD:R_0805_2012Metric"
 			(at 172.466 44.704 90)
 			(effects
@@
 			)
 		)
-		(property "Footprint" ""
+		(property "Footprint" "Connector_PinHeader_1.00mm:PinHeader_1x01_P1.00mm_Vertical"
 			(at 114.3 125.73 0)
 			(effects
@@
 			)
 		)
-		(property "Footprint" ""
+		(property "Footprint" "Resistor_SMD:R_0805_2012Metric"
 			(at 228.346 47.244 90)
 			(effects
@@
 			)
 		)
-		(property "Footprint" ""
+		(property "Footprint" "Connector_PinHeader_1.00mm:PinHeader_1x01_P1.00mm_Vertical"
 			(at 114.3 101.6 0)
 			(effects
@@
 			)
 		)
-		(property "Footprint" ""
+		(property "Footprint" "Connector_PinHeader_1.00mm:PinHeader_1x01_P1.00mm_Vertical"
 			(at 114.3 114.3 0)
 			(effects
@@
 			)
 		)
-		(property "Footprint" ""
+		(property "Footprint" "Resistor_SMD:R_0805_2012Metric"
 			(at 122.936 45.974 90)
 			(effects

Commit message: Work done on 11/06/2024
Connections:
- net 24V renamed 48V
- net 24V_GND renamed 48V_GND
Other:
- note added: "48V LED"
- note removed: "24V LED"
Changed lines of the file:
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@@
 		)
 	)
-	(text "24V LED"
+	(text "48V LED"
 		(exclude_from_sim no)
 		(at 231.14 20.574 0)
@@
 		)
 	)
-	(global_label "24V"
+	(global_label "48V"
 		(shape input)
 		(at 31.75 113.03 180)
@@
 		)
 	)
-	(global_label "24V"
+	(global_label "48V"
 		(shape input)
 		(at 109.22 125.73 180)
@@
 		)
 	)
-	(global_label "24V"
+	(global_label "48V"
 		(shape input)
 		(at 237.49 25.4 0)
@@
 		)
 	)
-	(global_label "24V_GND"
+	(global_label "48V_GND"
 		(shape input)
 		(at 31.75 116.84 180)
@@
 		)
 	)
-	(global_label "24V_GND"
+	(global_label "48V_GND"
 		(shape input)
 		(at 109.22 132.08 180)
@@
 		)
 	)
-	(global_label "24V_GND"
+	(global_label "48V_GND"
 		(shape input)
 		(at 237.49 55.88 0)

Commit message: Work done on 11/22/2024
Parts:
- C2, C5: footprint Capacitor_SMD:C_0805_2012Metric -> EEE_FT1E561UPfootprints:CAP_FT_F_PAN
- J10, J11, J13, J15, J16, J6, J7, J9: footprint Connector_PinHeader_1.00mm:PinHeader_1x01_P1.00mm_Vertical -> TestPoint:TestPoint_Pad_D4.0mm
- R5, R6, R7, R8: footprint Resistor_SMD:R_0805_2012Metric -> Resistor_SMD:R_0603_1608Metric
Changed lines of the file:
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@@
 			)
 		)
-		(property "Footprint" "Connector_PinHeader_1.00mm:PinHeader_1x01_P1.00mm_Vertical"
+		(property "Footprint" "TestPoint:TestPoint_Pad_D4.0mm"
 			(at 114.3 107.95 0)
 			(effects
@@
 			)
 		)
-		(property "Footprint" "Capacitor_SMD:C_0805_2012Metric"
+		(property "Footprint" "EEE_FT1E561UPfootprints:CAP_FT_F_PAN"
 			(at 44.45 39.37 0)
 			(effects
@@
 			)
 		)
-		(property "Footprint" "Connector_PinHeader_1.00mm:PinHeader_1x01_P1.00mm_Vertical"
+		(property "Footprint" "TestPoint:TestPoint_Pad_D4.0mm"
 			(at 114.3 95.25 0)
 			(effects
@@
 			)
 		)
-		(property "Footprint" "Connector_PinHeader_1.00mm:PinHeader_1x01_P1.00mm_Vertical"
+		(property "Footprint" "TestPoint:TestPoint_Pad_D4.0mm"
 			(at 114.3 119.38 0)
 			(effects
@@
 			)
 		)
-		(property "Footprint" "Capacitor_SMD:C_0805_2012Metric"
+		(property "Footprint" "EEE_FT1E561UPfootprints:CAP_FT_F_PAN"
 			(at 30.48 39.37 0)
 			(effects
@@
 			)
 		)
-		(property "Footprint" "Connector_PinHeader_1.00mm:PinHeader_1x01_P1.00mm_Vertical"
+		(property "Footprint" "TestPoint:TestPoint_Pad_D4.0mm"
 			(at 114.3 88.9 0)
 			(effects
@@
 			)
 		)
-		(property "Footprint" "Connector_PinHeader_1.00mm:PinHeader_1x01_P1.00mm_Vertical"
+		(property "Footprint" "TestPoint:TestPoint_Pad_D4.0mm"
 			(at 114.3 132.08 0)
 			(effects
@@
 			)
 		)
-		(property "Footprint" "Resistor_SMD:R_0805_2012Metric"
+		(property "Footprint" "Resistor_SMD:R_0603_1608Metric"
 			(at 94.996 44.704 90)
 			(effects
@@
 			)
 		)
-		(property "Footprint" "Resistor_SMD:R_0805_2012Metric"
+		(property "Footprint" "Resistor_SMD:R_0603_1608Metric"
 			(at 172.466 44.704 90)
 			(effects
@@
 			)
 		)
-		(property "Footprint" "Connector_PinHeader_1.00mm:PinHeader_1x01_P1.00mm_Vertical"
+		(property "Footprint" "TestPoint:TestPoint_Pad_D4.0mm"
 			(at 114.3 125.73 0)
 			(effects
@@
 			)
 		)
-		(property "Footprint" "Resistor_SMD:R_0805_2012Metric"
+		(property "Footprint" "Resistor_SMD:R_0603_1608Metric"
 			(at 228.346 47.244 90)
 			(effects
@@
 			)
 		)
-		(property "Footprint" "Connector_PinHeader_1.00mm:PinHeader_1x01_P1.00mm_Vertical"
+		(property "Footprint" "TestPoint:TestPoint_Pad_D4.0mm"
 			(at 114.3 101.6 0)
 			(effects
@@
 			)
 		)
-		(property "Footprint" "Connector_PinHeader_1.00mm:PinHeader_1x01_P1.00mm_Vertical"
+		(property "Footprint" "TestPoint:TestPoint_Pad_D4.0mm"
 			(at 114.3 114.3 0)
 			(effects
@@
 			)
 		)
-		(property "Footprint" "Resistor_SMD:R_0805_2012Metric"
+		(property "Footprint" "Resistor_SMD:R_0603_1608Metric"
 			(at 122.936 45.974 90)
 			(effects
